Commit message: Fix raw ptr usage. Increase support for non pointmass robots

File: src/goc_mpc/descriptions/point_mass_3dof.urdf (robot description, URDF)
Before this commit: robot point_mass_3dof, 3 links, 3 joints
Links:
- removed link pm_body
- added link ee_link, mass 1.0; collision sphere radius=0.02; visual sphere radius=0.02
Joints:
- joint jz: child pm_body -> ee_link
