Commit message: Change initial robot orientation to match reality

File: src/goc_mpc/descriptions/free_body_6dof.urdf (robot description, URDF)
Before this commit: robot free_body_6dof_actuated, 1 links, 1 joints
Links:
- link ee_link: geometry collision sphere radius=0.06; visual box size=0.06 0.03 0.06
